File: Hardware/IceFlow/IceFlow.kicad_sch (KiCad schematic)
At the start: 24 parts, among them J1 Barrel_Jack_Switch, J2 Conn_01x04, J3 TFT_Display_wTouch, J4 SSR_Oven, J5 SSR_Fan, J6 TempProbe_A, J7 TempProbe_A, J8 Power_Sw, U1 NCP1117-3.3_SOT223, U2 ESP32-WROVER-E

Commit message: PCB Updates
Parts:
- removed J4: SSR_Oven, Connector_PinHeader_2.54mm:PinHeader_1x02_P2.54mm_Vertical, symbol Connector_Generic:Conn_01x02
- removed J5: SSR_Fan, Connector_PinHeader_2.54mm:PinHeader_1x02_P2.54mm_Vertical, symbol Connector_Generic:Conn_01x02
- removed J6, J7: TempProbe_A, Connector_PinHeader_2.54mm:PinHeader_1x05_P2.54mm_Vertical, symbol Connector_Generic:Conn_01x05
- added J4: Conn_02x02_Odd_Even, Connector_PinHeader_2.54mm:PinHeader_2x02_P2.54mm_Horizontal, symbol Connector_Generic:Conn_02x02_Odd_Even
- added J6: Conn_02x05_Odd_Even, Connector_PinHeader_2.54mm:PinHeader_2x05_P2.54mm_Horizontal, symbol Connector_Generic:Conn_02x05_Odd_Even
- H1, H2, H3, H4: footprint MountingHole:MountingHole_2.7mm_M2.5_DIN965 -> MountingHole:MountingHole_3.2mm_M3_DIN965
- J2: footprint Connector_PinHeader_2.54mm:PinHeader_1x04_P2.54mm_Vertical -> Connector_PinHeader_2.54mm:PinHeader_1x04_P2.54mm_Horizontal
- J8: footprint Connector_PinHeader_2.54mm:PinHeader_1x02_P2.54mm_Vertical -> Connector_PinHeader_2.54mm:PinHeader_1x02_P2.54mm_Horizontal
Connections:
- net +3V3: now also J2.2 (Pin_2), J6.10 (Pin_10), J6.9 (Pin_9); no longer J2.3 (Pin_3)
- net CLK: now also J6.1 (Pin_1), J6.2 (Pin_2)
- net DO: now also J6.5 (Pin_5), J6.6 (Pin_6)
- net GND: now also J2.1 (Pin_1), J4.1 (Pin_1), J4.2 (Pin_2), J6.7 (Pin_7), J6.8 (Pin_8); no longer J2.4 (Pin_4)
- net SSR_F: now also J4.3 (Pin_3)
- net SSR_O: now also J4.4 (Pin_4)
- net TPA_CS: now also J6.4 (Pin_4)
- net TPB_CS: now also J6.3 (Pin_3)
- net Vin: now also J8.2 (Pin_2); no longer J8.1 (Pin_1)
- net at J1.1: now also J8.1 (Pin_1); no longer J8.2 (Pin_2)
- net at U2.35 (U0TXD/GPIO1): now also J2.4 (Pin_4); no longer J2.1 (Pin_1)
- net at U2.34 (U0RXD/GPIO3): now also J2.3 (Pin_3); no longer J2.2 (Pin_2)
Other:
- moved on the sheet: J2, J8
