File: Hardware/IceFlow/IceFlow.kicad_sch (KiCad schematic)
At the start: 23 parts, among them J1 Barrel_Jack_Switch, J2 Conn_01x04, J3 TFT_Display_wTouch, J4 Conn_02x02_Odd_Even, J5 USB_MICRO-B_SMT, J6 Conn_02x05_Odd_Even, J8 Power_Sw, U1 NCP1117-3.3_SOT223, U2 ESP32-WROVER-E

Commit message: Pin map changes
Parts:
- D1: footprint LED_SMD:LED_0805_2012Metric_Pad1.15x1.40mm_HandSolder -> LED_SMD:LED_1206_3216Metric_Pad1.42x1.75mm_HandSolder
- R2: footprint Resistor_SMD:R_0805_2012Metric_Pad1.20x1.40mm_HandSolder -> Resistor_SMD:R_1206_3216Metric_Pad1.30x1.75mm_HandSolder
Changed lines of the file:
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@@
     (property "Reference" "D1" (id 0) (at 48.5775 138.2862 0))
     (property "Value" "LED" (id 1) (at 48.5775 140.8231 0))
-    (property "Footprint" "LED_SMD:LED_0805_2012Metric_Pad1.15x1.40mm_HandSolder" (id 2) (at 46.99 144.145 0)
+    (property "Footprint" "LED_SMD:LED_1206_3216Metric_Pad1.42x1.75mm_HandSolder" (id 2) (at 46.99 144.145 0)
       (effects (font (size 1.27 1.27)) hide)
     )
@@
     (property "Reference" "R2" (id 0) (at 34.29 142.875 90))
     (property "Value" "64.9R" (id 1) (at 40.005 142.875 90))
-    (property "Footprint" "Resistor_SMD:R_0805_2012Metric_Pad1.20x1.40mm_HandSolder" (id 2) (at 37.465 144.145 0)
+    (property "Footprint" "Resistor_SMD:R_1206_3216Metric_Pad1.30x1.75mm_HandSolder" (id 2) (at 37.465 144.145 0)
       (effects (font (size 1.27 1.27)) hide)
     )
@@
     )
     (path "/2460d235-2c76-4e55-b43b-69ba996c31c9"
-      (reference "D1") (unit 1) (value "LED") (footprint "LED_SMD:LED_0805_2012Metric_Pad1.15x1.40mm_HandSolder")
+      (reference "D1") (unit 1) (value "LED") (footprint "LED_SMD:LED_1206_3216Metric_Pad1.42x1.75mm_HandSolder")
     )
     (path "/b06ecf3c-0e3f-4017-bb6d-0a3c37b098e1"
@@
     )
     (path "/571b50bb-72aa-441a-a0e3-b564c0d0e486"
-      (reference "R2") (unit 1) (value "64.9R") (footprint "Resistor_SMD:R_0805_2012Metric_Pad1.20x1.40mm_HandSolder")
+      (reference "R2") (unit 1) (value "64.9R") (footprint "Resistor_SMD:R_1206_3216Metric_Pad1.30x1.75mm_HandSolder")
     )
     (path "/a2d00796-078f-401b-983d-8b8112e5c730"
