File: Hardware/IceFlow/IceFlow.kicad_pcb (KiCad board)
At the start: 2 copper layers, 63.5 x 36.2 mm, 24 parts, among them J1 Barrel_Jack_Switch, J2 Conn_01x04, J3 TFT_Display_wTouch, J4 SSR_Oven, J5 SSR_Fan, J6 TempProbe_A, J7 TempProbe_A, J8 Power_Sw, U1 NCP1117-3.3_SOT223, U2 ESP32-WROVER-E

Commit message: PCB Updates
Parts:
- removed J5: SSR_Fan, Connector_PinHeader_2.54mm:PinHeader_1x02_P2.54mm_Vertical
- removed J7: TempProbe_A, Connector_PinHeader_2.54mm:PinHeader_1x05_P2.54mm_Vertical
- H1, H2, H3, H4: footprint MountingHole:MountingHole_2.7mm_M2.5_DIN965 -> MountingHole:MountingHole_3.2mm_M3_DIN965
- J2: footprint Connector_PinHeader_2.54mm:PinHeader_1x04_P2.54mm_Vertical -> Connector_PinHeader_2.54mm:PinHeader_1x04_P2.54mm_Horizontal
- J4: value SSR_Oven -> Conn_02x02_Odd_Even; footprint Connector_PinHeader_2.54mm:PinHeader_1x02_P2.54mm_Vertical -> Connector_PinHeader_2.54mm:PinHeader_2x02_P2.54mm_Horizontal
- J6: value TempProbe_A -> Conn_02x05_Odd_Even; footprint Connector_PinHeader_2.54mm:PinHeader_1x05_P2.54mm_Vertical -> Connector_PinHeader_2.54mm:PinHeader_2x05_P2.54mm_Horizontal
- J8: footprint Connector_PinHeader_2.54mm:PinHeader_1x02_P2.54mm_Vertical -> Connector_PinHeader_2.54mm:PinHeader_1x02_P2.54mm_Horizontal
- moved J4 20.2 mm to (83.2, 123.2), turned to -90 degrees
- moved H1 19.8 mm to (68.7, 81.3)
- moved H3 15.8 mm to (145.3, 81.3)
- moved H2 13.8 mm to (68.7, 124.7)
- moved J6 10.8 mm to (113.0, 121.4), turned to -90 degrees
- moved J2 7.76 mm to (124.5, 124.1), turned to -90 degrees
- moved H4 6.86 mm to (145.3, 124.7)
- moved J8 3.41 mm to (90.8, 116.2), turned to 180 degrees
- moved C1 2.41 mm to (95.9, 114.3)
- moved S1 1.33 mm to (101.0, 105.4)
Connections:
- J1 pad 1: Net-(J8-Pad2) -> Net-(J1-Pad1)
- J2 pad 1: Net-(J2-Pad1) -> GND
- J2 pad 2: Net-(J2-Pad2) -> +3V3
- J2 pad 3: +3V3 -> Net-(U2-Pad34)
- J2 pad 4: GND -> Net-(U2-Pad35)
- J4 pad 2: /SSR_O -> GND
- J6 pad 1: +3V3 -> /CLK
- J6 pad 2: GND -> /CLK
- J6 pad 3: /DO -> /TPB_CS
- J6 pad 5: /CLK -> /DO
- J8 pad 1: /Vin -> Net-(J1-Pad1)
- J8 pad 2: Net-(J8-Pad2) -> /Vin
- U2 pad 34: Net-(J2-Pad2) -> Net-(U2-Pad34)
- U2 pad 35: Net-(J2-Pad1) -> Net-(U2-Pad35)
Routing:
- net /SSR_F: track 10.5 -> 51.6 mm, vias 0 -> 2
- net /SSR_O: track 12.6 -> 48.9 mm, vias 0 -> 2
- net Net-(J2-Pad1): track 34.1 -> 0.00 mm
- net Net-(U2-Pad35): track 0.00 -> 32.5 mm
- net Net-(J2-Pad2): track 32.1 -> 0.00 mm
- net Net-(U2-Pad34): track 0.00 -> 30.5 mm
- net GND: track 41.8 -> 28.9 mm, vias 8 -> 7
- net /TPA_CS: track 26.3 -> 32.8 mm, vias 1 -> 2
- net /EN: track 15.8 -> 17.3 mm
- net /CLK: track 23.2 -> 21.9 mm
- net /DO: track 19.9 -> 18.7 mm
- net +3V3: track 104.9 -> 105.7 mm
- net /MOSI: track 22.7 -> 21.9 mm
- net /Rst: track 16.1 -> 15.3 mm
- net /D/C: track 14.8 -> 14.0 mm
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- added copper zone on F.Cu, net GND
- added copper zone on F.Cu, net Net-(J1-Pad1)
- removed copper zone on F.Cu, net Net-(J8-Pad2)
Other:
- board size 63.5 x 36.2 mm -> 84 x 52.5 mm
- board text added: "Fan --- Oven"
- board text added: "Gnd"
- board text added: "Kitecraft"
- board text added: "Relays"
- board text added: "Signal"
- board text added: "Temp Probes Primary Secondary"
- board text added: "V 1.0"
- board text removed: "Gnd Sig"
- board text removed: "Oven Fan"
- board text removed: "Temp Probes One Two"

Commit message: PCB Update
Routing:
- net /TPA_CS: track 32.8 -> 28.1 mm
Changed lines of the file:
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@@
   (via (at 123.952 111.379) (size 0.8) (drill 0.4) (layers "F.Cu" "B.Cu") (net 31))
   (via (at 118.618 111.506) (size 0.8) (drill 0.4) (layers "F.Cu" "B.Cu") (net 31))
-  (segment (start 123.952 111.379) (end 119.253 111.379) (width 0.25) (layer "B.Cu") (net 31))
   (segment (start 123.825 111.506) (end 123.952 111.379) (width 0.25) (layer "B.Cu") (net 31))
   (segment (start 118.618 111.506) (end 123.825 111.506) (width 0.25) (layer "B.Cu") (net 31))
